File: kicad/board/board.kicad_pcb (KiCad board)
At the start: 2 copper layers, 126.9 x 103.7 mm, 39 parts

Commit message: Clacken w/ Completed Schematic
Parts:
- added H1: MountingHole, MountingHole:MountingHole_2.2mm_M2, F.Cu at (99.3, 35.1)
- added H2: MountingHole, MountingHole:MountingHole_2.2mm_M2, F.Cu at (75.8, -31.6)
- added H3: MountingHole, MountingHole:MountingHole_2.2mm_M2, F.Cu at (0.00, 5.50)
- added H4: MountingHole, MountingHole:MountingHole_2.2mm_M2, F.Cu at (0.00, -30.5)
- added S19: SSSS811101, onOffFootprint:SW_SSSS811101, B.Cu at (103.0, -1.50)
- added S20: SSSS811101, onOffFootprint:SW_SSSS811101, F.Cu at (103.0, -1.50)
- D1, D10, D11, D12, D13, D14, D15, D16, D17, D18, D2, D3, D4, D5, D6, D7, D8, D9: value 1N914 -> 1N4001; footprint clacken:reversable_diode -> clackenFootprints:reversable_diode
- JST1, JST2: footprint clacken:JST_angled -> clackenFootprints:JST_angled
- S1, S10, S11, S12, S13, S14, S15, S16, S17, S18, S2, S3, S4, S5, S6, S7, S8, S9: value SW_Push_45deg -> SW_SPST; footprint clacken:choc_switches -> clackenFootprints:choc_switches
- U1: value (none) -> ~; footprint xiao-ble-tht -> clackenFootprints:seeed_xaio
Connections:
- D1 pad 1: Row3 -> Net-(D1-K)
- D10 pad 1: Row3 -> Net-(D1-K)
- D11 pad 1: Row2 -> Net-(D11-K)
- D12 pad 1: Row1 -> Net-(D12-K)
- D13 pad 1: Row3 -> Net-(D1-K)
- D14 pad 1: Row2 -> Net-(D11-K)
- D15 pad 1: Row1 -> Net-(D12-K)
- D16 pad 1: Row4 -> Net-(D16-K)
- D17 pad 1: Row4 -> Net-(D16-K)
- D18 pad 1: Row4 -> Net-(D16-K)
- D2 pad 1: Row2 -> Net-(D11-K)
- D3 pad 1: Row1 -> Net-(D12-K)
- D4 pad 1: Row3 -> Net-(D1-K)
- D5 pad 1: Row2 -> Net-(D11-K)
- D6 pad 1: Row1 -> Net-(D12-K)
- D7 pad 1: Row3 -> Net-(D1-K)
- D8 pad 1: Row2 -> Net-(D11-K)
- D9 pad 1: Row1 -> Net-(D12-K)
- JST2 pad 2: Net-(JST1-Pin_2) -> Net-(JST2-Pin_2)
- S1 pad 1: Col1 -> Net-(S1-A)
- S10 pad 1: Col4 -> Net-(S10-A)
- S11 pad 1: Col4 -> Net-(S10-A)
- S12 pad 1: Col4 -> Net-(S10-A)
- S13 pad 1: Col5 -> Net-(S13-A)
- S14 pad 1: Col5 -> Net-(S13-A)
- S15 pad 1: Col5 -> Net-(S13-A)
- S16 pad 1: Col3 -> Net-(S16-A)
- S17 pad 1: Col4 -> Net-(S10-A)
- S18 pad 1: Col5 -> Net-(S13-A)
- S2 pad 1: Col1 -> Net-(S1-A)
- S3 pad 1: Col1 -> Net-(S1-A)
- S4 pad 1: Col2 -> Net-(S4-A)
- S5 pad 1: Col2 -> Net-(S4-A)
- S6 pad 1: Col2 -> Net-(S4-A)
- S7 pad 1: Col3 -> Net-(S16-A)
- S8 pad 1: Col3 -> Net-(S16-A)
- S9 pad 1: Col3 -> Net-(S16-A)
- U1 pad 0: P0 -> Net-(S1-A)
- U1 pad 1: P1 -> Net-(S4-A)
- U1 pad 10: P10 -> unconnected-(U1-P10-Pad10)
- U1 pad 11: _1_11 -> unconnected-(U1-V3-Pad11)
- U1 pad 12: _1_12 -> unconnected-(U1-GND-Pad12)
- U1 pad 13: _1_13 -> unconnected-(U1-VCC-Pad13)
- U1 pad 2: P2 -> Net-(S16-A)
- U1 pad 3: P3 -> Net-(S10-A)
- U1 pad 4: P4 -> Net-(D12-K)
- U1 pad 5: P5 -> Net-(D11-K)
- U1 pad 6: P6 -> Net-(D1-K)
- U1 pad 7: P7 -> Net-(D16-K)
- U1 pad 8: P8 -> Net-(S13-A)
- U1 pad 9: P9 -> unconnected-(U1-P9-Pad9)
Routing:
- net (no net): track 0.00 -> 24.0 mm
- net unconnected-(U1-VCC-Pad13): track 0.00 -> 10.3 mm
- net VCC: track 10.3 -> 0.00 mm
- net unconnected-(U1-GND-Pad12): track 0.00 -> 10.3 mm
- net P0: track 10.3 -> 0.00 mm
- net Net-(S1-A): track 0.00 -> 10.3 mm
- net GND: track 10.3 -> 0.00 mm
- net unconnected-(U1-V3-Pad11): track 0.00 -> 10.3 mm
- net V3: track 10.3 -> 0.00 mm
- net P1: track 10.3 -> 0.00 mm
- net Net-(S4-A): track 0.00 -> 10.3 mm
- net P2: track 10.3 -> 0.00 mm
- net Net-(S16-A): track 0.00 -> 10.3 mm
- net _1_12: track 4.01 -> 0.00 mm
- net _1_1: track 4.01 -> 0.00 mm
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