File: kicad/board/board.kicad_pcb (KiCad board)
At the start: 2 copper layers, 126.9 x 103.7 mm, 45 parts

Commit message: Keyboard with Traces
Parts:
- moved S19 0.50 mm to (102.5, -1.50)
- moved S20 0.50 mm to (102.5, -1.50)
Routing:
- net Net-(S16-A): track 10.3 -> 202.7 mm, vias 0 -> 6
- net Net-(S10-A): track 0.00 -> 189.7 mm, vias 0 -> 4
- net Net-(S1-A): track 10.3 -> 179.2 mm, vias 0 -> 3
- net Net-(S13-A): track 0.00 -> 152.3 mm, vias 0 -> 5
- net Net-(S4-A): track 10.3 -> 162.2 mm, vias 0 -> 4
- net Net-(D16-K): track 0.00 -> 139.8 mm
- net Net-(D1-K): track 0.00 -> 127.4 mm
- net Net-(D11-K): track 0.00 -> 111.5 mm
- net Net-(D12-K): track 0.00 -> 96.7 mm
- net Net-(D2-A): track 0.00 -> 36.8 mm
- net Net-(D16-A): track 0.00 -> 28.5 mm
- net Net-(D6-A): track 0.00 -> 28.2 mm
- net Net-(JST1-Pin_2): track 0.00 -> 28.2 mm, vias 0 -> 1
- net Net-(D12-A): track 0.00 -> 28.1 mm
- net Net-(D10-A): track 0.00 -> 28.0 mm
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
Commit message: fixed wiring
Routing:
- net Net-(D11-A): track 20.9 -> 27.8 mm
Changed lines of the file:
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@@
 			(outputformat 1)
 			(mirror no)
-			(drillshape 1)
+			(drillshape 0)
 			(scaleselection 1)
-			(outputdirectory "")
+			(outputdirectory "gerber/")
 		)
 	)
@@
 		)
 		(pad "2" thru_hole circle
-			(at -3.262003 -2.54)
+			(at -3.262004 -2.54)
 			(size 0.8 0.8)
 			(drill 0.4)
@@
 		(fp_line
 			(start 3.35 0.379999)
-			(end 3.350001 -0.380001)
+			(end 3.350002 -0.380001)
 			(stroke
 				(width 0.127)
@@
 		)
 		(fp_line
-			(start -3.350001 0.380001)
+			(start -3.350002 0.380001)
 			(end -3.35 -0.379999)
 			(stroke
@@
 		(net 11)
 	)
+	(segment
+		(start 65.525297 -21.380914)
+		(end 63.682293 -19.53791)
+		(width 0.25)
+		(layer "B.Cu")
+		(net 11)
+	)
+	(segment
+		(start 65.525297 -25.694049)
+		(end 65.525297 -21.380914)
+		(width 0.25)
+		(layer "B.Cu")
+		(net 11)
+	)
